Commit message: add gazebo simulation

File: eleven_description/urdf/eleven_base.xacro (robot description, xacro)
@@ -5,16 +5,86 @@
     <xacro:include filename="$(find anman_sensors)/sensors/imu_mpu9250/imu_mpu9250.xacro"/>
     <xacro:include filename="$(find anman_sensors)/sensors/ydlidar/ydlidar_g4.xacro"/>
+    <xacro:include filename="$(find anman_sensors)/actuators/bldc_hover_65/bldc_hover_65.xacro"/>
     <link name="base_footprint"/>
     <joint name="base_fixed" type="fixed">
-        <origin xyz="0 0 0.2" rpy="0 0 0"/>
+        <origin xyz="0 0 0.1" rpy="0 0 0"/>
         <parent link="base_footprint"/>
         <child link="base_link"/>
     </joint>
-    <link name="base_link"/>
-    <imu_mpu9250 prefix="imu" parent="base_link">
-        <origin xyz="-0.2 0 0" rpy="0 0 0"/>
-    </imu_mpu9250>
-    <ydlidar_g4 prefix="laser" parent="base_link" min_angle="-1.570796" max_angle="1.570796" prefix_topic=''>
-        <origin xyz="0.1 0 0.1" rpy="0 0 0"/>
-    </ydlidar_g4>
+    <link name="base_link">
+        <visual>
+            <origin xyz="0 0 -0.055" rpy="1.5707 0 -1.5707" />
+            <geometry>
+                <mesh filename="package://eleven_description/meshes/chessis.STL" scale="1 1 1" />
+            </geometry>
+            <material name="green"/>
+        </visual>
+        <collision name="chessis_collision">
+            <origin xyz="0 0 -0.055" rpy="1.5707 0 -1.5707" />
+            <geometry>
+                <mesh filename="package://eleven_description/meshes/chessis.STL" scale="1 1 1" />
+            </geometry>
+            <surface>
+                <friction>
+                    <ode>
+                        <mu>0.1</mu>
+                        <mu2>0.1</mu2>
+                        <slip1>1.0</slip1>
+                        <slip2>1.0</slip2>
+                    </ode>
+                </friction>
+            </surface>
+        </collision>
+        <inertial>
+            <mass value="10.0"/>
+            <origin xyz="-0.2 0 0.1" rpy=" 0 0 0"/>
+            <inertia ixx="0.1" ixy="0" ixz="0" iyy="0.1" iyz="0" izz="0.1" />
+        </inertial>
+    </link>
+    <gazebo reference="base_link">
+        <mu1>0.0001</mu1>
+        <mu2>0.0001</mu2>
+        <material>Gazebo/Red</material>
+    </gazebo>
+    <xacro:bldc_hover_65 prefix="left_wheel" parent="base_link" reflect="1">
+        <origin xyz="0 0.23 -0.02" rpy="0 ${PI/2} ${PI/2}"/>
+    </xacro:bldc_hover_65>
+    <xacro:bldc_hover_65 prefix="right_wheel" parent="base_link" reflect="-1">
+        <origin xyz="0 -0.23 -0.02" rpy="0 ${PI/2} ${-PI/2}"/>
+    </xacro:bldc_hover_65>
+    <xacro:imu_mpu9250 prefix="imu" parent="base_link">
+        <origin xyz="-0.25 0.08 0.1" rpy="0 0 ${PI/2}"/>
+    </xacro:imu_mpu9250>
+    <xacro:ydlidar_g4 prefix="laser" parent="base_link" min_angle="-1.570796" max_angle="1.570796" prefix_topic='eleven'>
+        <origin xyz="0.15 0 0.1" rpy="0 0 0"/>
+    </xacro:ydlidar_g4>
+    <gazebo>
+        <plugin name="differential_drive_controller" filename="libgazebo_ros_diff_drive.so">
+            <!-- <robotNamespace></robotNamespace> -->
+            <alwaysOn>true</alwaysOn>
+            <updateRate>20</updateRate>
+            <leftJoint>left_wheel_joint</leftJoint>
+            <rightJoint>right_wheel_joint</rightJoint>
+            <wheelSeparation>0.46</wheelSeparation>
+            <wheelDiameter>0.1651</wheelDiameter>
+            <wheelTorque>20</wheelTorque>
+            <commandTopic>eleven/cmd_vel</commandTopic>
+            <odometryTopic>eleven/odom</odometryTopic>
+            <odometryFrame>odom</odometryFrame>
+            <robotBaseFrame>base_footprint</robotBaseFrame>
+            <legacyMode>false</legacyMode>
+            <publishOdomTF>true</publishOdomTF>
+            <rosDebugLevel>Debug</rosDebugLevel>
+            <publishWheelTF>true</publishWheelTF>
+            <publishWheelJointState>false</publishWheelJointState>
+            <wheelAcceleration>5</wheelAcceleration>
+            <publishTf>1</publishTf>
+            <odometrySource>encoder</odometrySource>
+        </plugin>
+        <plugin name="gazebo_ros_control" filename="libgazebo_ros_control.so">
+            <robotNamespace>/eleven</robotNamespace>
+            <robotParam>/robot_description</robotParam>
+            <robotSimType>gazebo_ros_control/DefaultRobotHWSim</robotSimType>
+        </plugin>
+    </gazebo>
 </robot>

Commit message: update simulation

File: eleven_description/urdf/eleven_base.xacro (robot description, xacro)
@@ -38,6 +38,7 @@
         <inertial>
             <mass value="10.0"/>
-            <origin xyz="-0.2 0 0.1" rpy=" 0 0 0"/>
-            <inertia ixx="0.1" ixy="0" ixz="0" iyy="0.1" iyz="0" izz="0.1" />
+            <origin xyz="-0.15 0 0.1" rpy=" 0 0 0"/>
+            <!-- <inertia ixx="0.1" ixy="0" ixz="0" iyy="0.1" iyz="0" izz="0.1" /> -->
+            <xacro:box_inertia m="10.0" x="0.4" y="0.4" z="0.2"/>
         </inertial>
     </link>
@@ -53,13 +54,12 @@
         <origin xyz="0 -0.23 -0.02" rpy="0 ${PI/2} ${-PI/2}"/>
     </xacro:bldc_hover_65>
-    <xacro:imu_mpu9250 prefix="imu" parent="base_link">
+    <xacro:imu_mpu9250 prefix="imu" parent="base_link" prefix_topic=''>
         <origin xyz="-0.25 0.08 0.1" rpy="0 0 ${PI/2}"/>
     </xacro:imu_mpu9250>
-    <xacro:ydlidar_g4 prefix="laser" parent="base_link" min_angle="-1.570796" max_angle="1.570796" prefix_topic='eleven'>
+    <xacro:ydlidar_g4 prefix="laser" parent="base_link" prefix_topic='' min_angle="-1.570796" max_angle="1.570796" min_range="0.26" max_range="12.0">
         <origin xyz="0.15 0 0.1" rpy="0 0 0"/>
     </xacro:ydlidar_g4>
     <gazebo>
         <plugin name="differential_drive_controller" filename="libgazebo_ros_diff_drive.so">
-            <!-- <robotNamespace></robotNamespace> -->
             <alwaysOn>true</alwaysOn>
             <updateRate>20</updateRate>
@@ -69,21 +69,21 @@
             <wheelDiameter>0.1651</wheelDiameter>
             <wheelTorque>20</wheelTorque>
-            <commandTopic>eleven/cmd_vel</commandTopic>
-            <odometryTopic>eleven/odom</odometryTopic>
+            <commandTopic>cmd_vel</commandTopic>
+            <odometryTopic>odom_wheel</odometryTopic>
             <odometryFrame>odom</odometryFrame>
             <robotBaseFrame>base_footprint</robotBaseFrame>
-            <legacyMode>false</legacyMode>
-            <publishOdomTF>true</publishOdomTF>
-            <rosDebugLevel>Debug</rosDebugLevel>
-            <publishWheelTF>true</publishWheelTF>
+            <!-- <rosDebugLevel>Debug</rosDebugLevel> -->
+            <rosDebugLevel>na</rosDebugLevel>
+            <publishWheelTF>false</publishWheelTF>
             <publishWheelJointState>false</publishWheelJointState>
-            <wheelAcceleration>5</wheelAcceleration>
+            <publishOdomTF>false</publishOdomTF>
+            <wheelAcceleration>0</wheelAcceleration>
             <publishTf>1</publishTf>
             <odometrySource>encoder</odometrySource>
         </plugin>
         <plugin name="gazebo_ros_control" filename="libgazebo_ros_control.so">
-            <robotNamespace>/eleven</robotNamespace>
+            <!-- <robotNamespace>/eleven</robotNamespace> -->
             <robotParam>/robot_description</robotParam>
-            <robotSimType>gazebo_ros_control/DefaultRobotHWSim</robotSimType>
+            <!-- <robotSimType>gazebo_ros_control/DefaultRobotHWSim</robotSimType> -->
         </plugin>
     </gazebo>

Commit message: update slam

File: eleven_description/urdf/eleven_base.xacro (robot description, xacro)
@@ -57,6 +57,7 @@
         <origin xyz="-0.25 0.08 0.1" rpy="0 0 ${PI/2}"/>
     </xacro:imu_mpu9250>
-    <xacro:ydlidar_g4 prefix="laser" parent="base_link" prefix_topic='' min_angle="-1.570796" max_angle="1.570796" min_range="0.26" max_range="12.0">
-        <origin xyz="0.15 0 0.1" rpy="0 0 0"/>
+    <!-- <xacro:ydlidar_g4 prefix="laser" parent="base_link" prefix_topic='' min_angle="-1.570796" max_angle="1.570796" min_range="0.26" max_range="12.0"> -->
+    <xacro:ydlidar_g4 prefix="laser" parent="base_link" prefix_topic='' min_range="0.26" max_range="12.0">
+        <origin xyz="0.15 0 0.2" rpy="0 0 0"/>
     </xacro:ydlidar_g4>
     <gazebo>
